Commit message: Major changes to gazebo_ros_dc_motor.cpp, now the plugin ignores current dynamic and calculates torque from voltage input and wheel speed. Now the test environment read the wheel params from params/test.yaml

File: xacro/dc_motor.xacro (robot description, xacro)
@@ -2,6 +2,5 @@
 <robot xmlns:xacro="http://www.ros.org/wiki/xacro">
 <xacro:macro name="dc_motor" params="motor_name parent_link child_link *origin *axis">
-  <!-- <xacro:property name="params_yaml" value="$(find gazebo_ros_motors)/params/dc_motor.yaml"/> -->
-  <xacro:property name="motor_param" value="${load_yaml(params_yaml)}"/>
+  <xacro:property name="motor_param" value="${xacro.load_yaml(params_yaml)}"/>
   <joint name="${motor_name}" type="continuous">
       <parent link="${parent_link}"/>
@@ -36,4 +35,5 @@
       <gear_ratio>${motor_param['gear_ratio']}</gear_ratio>
       <encoder_ppr>${motor_param['encoder_ppr']}</encoder_ppr>
+      <velocity_noise>${motor_param['velocity_noise']}</velocity_noise>
       <rosDebugLevel>Debug</rosDebugLevel>
     </plugin>

File: xacro/joint_motor.xacro (robot description, xacro)
@@ -3,5 +3,5 @@
 <xacro:macro name="joint_motor" params="motor_name parent_link child_link *origin *axis">
   <xacro:property name="params_yaml"  value="$(find gazebo_ros_motors)/params/joint_motor.yaml"/>
-  <xacro:property name="motor_param" value="${load_yaml(params_yaml)}"/>
+  <xacro:property name="motor_param" value="${xacro.load_yaml(params_yaml)}"/>
   <joint name="${motor_name}" type="continuous">
       <parent link="${parent_link}"/>

File: xacro/test.xacro (robot description, xacro)
@@ -1,4 +1,14 @@
 <?xml version="1.0"?>
 <robot name="motor" xmlns:xacro="http://www.ros.org/wiki/xacro">
+<!-- Include robot physical parameters -->
+<xacro:property name="wheel_params_file" value="$(find gazebo_ros_motors)/params/test.yaml"/>
+<xacro:property name="wheel_params" value="${xacro.load_yaml(wheel_params_file)}"/>
+<xacro:property name="wheel_name" value="one"/>
+<!-- Wheel Properties -->
+<xacro:property name="wheel_width" value="${wheel_params['wheel_width']}" />
+<xacro:property name="wheel_radius" value="${wheel_params['wheel_radius']}" />
+<xacro:property name="wheel_weight" value="${wheel_params['wheel_weight']}" />
+<!-- Inertial Properties -->
+<xacro:property name="wheel_I" value="${wheel_params['wheel_I']}" />
   <link name="base_footprint"/>
   <link name="base_link">
@@ -32,5 +42,5 @@
     <link name="${name}_wheel_link">
       <visual>
-        <origin rpy="0 0 0" xyz="0 0 0"/>
+        <origin rpy="0  0 0" xyz="0 0 0"/>
         <geometry>
             <cylinder length="0.05" radius="0.11"/>
@@ -46,26 +56,22 @@
         <origin rpy="0 0 0" xyz="0 0 0"/>
         <geometry>
-            <cylinder length="0.05" radius="0.11"/>
+			    <cylinder length="0.05" radius="0.11"/>
         </geometry>
-          <mass value="3.5"/>
-          <inertia ixx="0.0267" ixy="0" ixz="0" iyy="0.0267" iyz="0" izz="0.0506"/>
+        <!-- <mass value="1"/>
+        <inertia ixx="0.044" ixy="0" ixz="0" iyy="0.044" iyz="0" izz="0.001"/> -->
+        <mass value="${wheel_weight}" />
+        <inertia  ixx="${wheel_I['Ixx']}" ixy="${wheel_I['Ixy']}" ixz="${wheel_I['Ixz']}"
+					iyy="${wheel_I['Iyy']}" iyz="${wheel_I['Iyz']}"
+						izz="${wheel_I['Izz']}" />
       </inertial>
     </link>
   </xacro:macro>
-  <xacro:wheel name="one"/>
-  <!-- <xacro:wheel name="two"/>
-  <xacro:include filename="$(find gazebo_ros_motors)/xacro/joint_motor.xacro"/>
-  <xacro:joint_motor motor_name="one_motor" parent_link="base_link" child_link="one_wheel_link">
-    <xacro:property name="params_yaml" value="$(find gazebo_ros_motors)/params/joint_motor.yaml"/>
-    <origin xyz="0 0 0.2" rpy="0 0 0"/>
-  </xacro:joint_motor>
-  <xacro:joint_motor motor_name="two_motor" parent_link="base_link" child_link="two_wheel_link">
-    <xacro:property name="params_yaml" value="$(find gazebo_ros_motors)/params/joint_motor.yaml"/>
-    <origin xyz="0 0 0.4" rpy="0 0 0"/>
-  </xacro:joint_motor> -->
+  <xacro:wheel name="${wheel_name}"/>
   <xacro:include filename="$(find gazebo_ros_motors)/xacro/dc_motor.xacro"/>
-  <xacro:dc_motor motor_name="dc_motor" parent_link="base_link" child_link="one_wheel_link">
+  <xacro:dc_motor motor_name="${wheel_name}_wheel" parent_link="base_link" child_link="${wheel_name}_wheel_link">
     <xacro:property name="params_yaml" value="$(find gazebo_ros_motors)/params/dc_motor.yaml"/>
-    <origin xyz="0 0 0.2" rpy="0 0 0"/>
+    <!-- garantizo que la rueda no toque el suelo, elevandola mas alto que su radio -->
+    <origin xyz="0 0 ${wheel_radius*1.5}" rpy="1.5707 0 0"/>
+    <axis xyz="0 0 1" rpy="0 0 0"/>
   </xacro:dc_motor>
 </robot>
